File: PCB/majoras/majoras - rotate.kicad_pcb (KiCad board)
At the start: 2 copper layers, 13 x 6.5 mm, 13 parts

Commit message: Fabrication files for easy LED
Parts:
- removed the REF** at (145.0, 90.2) (x2)
- removed the REF** at (145.0, 91.8) (x2)
- removed the REF** at (154.5, 91.8) (x2)
- removed the REF** at (154.5, 88.8) (x2)
- removed the REF** at (154.5, 90.2) (x2)
- removed the REF** at (145.0, 88.8) (x2)
- added REF**: SolderWirePad_1x01_SMD_1x2mm, Connector_Wire:SolderWirePad_1x01_SMD_1x2mm, F.Cu at (165.8, 89.2)
- added REF**: SolderWirePad_1x01_SMD_1x2mm, Connector_Wire:SolderWirePad_1x01_SMD_1x2mm, B.Cu at (165.8, 89.2)
- added REF**: SolderWirePad_1x01_SMD_1x2mm, Connector_Wire:SolderWirePad_1x01_SMD_1x2mm, B.Cu at (159.2, 86.0)
- added REF**: SolderWirePad_1x01_SMD_1x2mm, Connector_Wire:SolderWirePad_1x01_SMD_1x2mm, B.Cu at (160.8, 86.0)
- added REF**: SolderWirePad_1x01_SMD_1x2mm, Connector_Wire:SolderWirePad_1x01_SMD_1x2mm, F.Cu at (160.8, 86.0)
- added REF**: SolderWirePad_1x01_SMD_1x2mm, Connector_Wire:SolderWirePad_1x01_SMD_1x2mm, F.Cu at (165.8, 90.8)
- added REF**: SolderWirePad_1x01_SMD_1x2mm, Connector_Wire:SolderWirePad_1x01_SMD_1x2mm, F.Cu at (165.8, 92.2)
- added REF**: SolderWirePad_1x01_SMD_1x2mm, Connector_Wire:SolderWirePad_1x01_SMD_1x2mm, F.Cu at (162.2, 86.0)
- added REF**: SolderWirePad_1x01_SMD_1x2mm, Connector_Wire:SolderWirePad_1x01_SMD_1x2mm, F.Cu at (159.2, 86.0)
- added REF**: SolderWirePad_1x01_SMD_1x2mm, Connector_Wire:SolderWirePad_1x01_SMD_1x2mm, B.Cu at (162.2, 86.0)
- added REF**: SolderWirePad_1x01_SMD_1x2mm, Connector_Wire:SolderWirePad_1x01_SMD_1x2mm, B.Cu at (165.8, 92.2)
- added REF**: SolderWirePad_1x01_SMD_1x2mm, Connector_Wire:SolderWirePad_1x01_SMD_1x2mm, B.Cu at (165.8, 90.8)
- moved D1 9.97 mm to (159.7, 91.8), turned to 45 degrees
Routing:
- net GND: track 16.5 -> 34.3 mm, vias 2 -> 0
- net DOUT: track 6.89 -> 13.6 mm, vias 2 -> 0
- net VDD: track 17.2 -> 19.5 mm, vias 2 -> 0
- net DIN: track 6.82 -> 7.57 mm, vias 2 -> 0
Other:
- board size 13 x 6.5 mm -> 10 x 10 mm

Commit message: Updated fabrication files
Parts:
- moved REF** 1.87 mm to (167.1, 90.6) (x2)
- moved REF** 1.87 mm to (167.1, 92.1) (x2)
- moved REF** 1.87 mm to (167.1, 93.6) (x2)
- moved REF** 1.03 mm to (158.8, 85.1) (x2)
- moved REF** 1.03 mm to (160.2, 85.1) (x2)
- moved REF** 1.03 mm to (161.8, 85.1) (x2)
- moved D1 0.85 mm to (160.6, 91.8)
Routing:
- net GND: track 34.3 -> 24.9 mm, vias 0 -> 4
- net DOUT: track 13.6 -> 7.45 mm, vias 0 -> 1
- net DIN: track 7.57 -> 5.71 mm, vias 0 -> 1
- net VDD: track 19.5 -> 18.4 mm, vias 0 -> 4
Other:
- board size 10 x 10 mm -> 11.8 x 11.8 mm
